File: dl3000-adapters.kicad_pcb (KiCad board)
At the start: 2 copper layers, 57 x 68 mm, 5 parts, among them J1 Banana Jack, J2 BNC, J3 Banana Jack

Commit message: Add information on bottom silk screen
Parts:
- added REF**: OSHW-Logo_5.7x6mm_SilkScreen, Symbol:OSHW-Logo_5.7x6mm_SilkScreen, B.Cu at (150.0, 51.5)
- added REF**: OSHW-Logo_5.7x6mm_SilkScreen, Symbol:OSHW-Logo_5.7x6mm_SilkScreen, B.Cu at (141.5, 100.0)
Other:
- board text added: "1.0"
- board text added: "DL3000 BNC Adapter"
- board text added: "DL3000 Banana Jack Adapter"
- board text added: "github.com/sirhcel/dl3000-adapters"
