File: dl3000-adapters.kicad_pcb (KiCad board)
At the start: 2 copper layers, 57 x 68 mm, 9 parts, among them J1 Banana Jack, J2 BNC, J3 Banana Jack

Commit message: Bump silk screen version to 1.1
Other:
- board text added: "1.1"
- board text removed: "1.0"
Changed lines of the file:
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@@
-(kicad_pcb (version 20171130) (host pcbnew "(5.1.8)-1")
+(kicad_pcb (version 20171130) (host pcbnew "(5.1.8-0-10_14)")
   (general
     (thickness 1.6)
@@
       (effects (font (size 1 1) (thickness 0.15)))
     )
-    (fp_text user "PCB Edge" (at 0 -2 90) (layer Dwgs.User)
-      (effects (font (size 1 1) (thickness 0.15)))
-    )
     (fp_line (start 3.75 -0.95) (end 3.75 16.05) (layer F.Fab) (width 0.1))
     (fp_line (start -3.75 -2.95) (end -3.75 -1.95) (layer F.Fab) (width 0.1))
@@
     (fp_line (start 3.75 17.05) (end 4.25 17.05) (layer F.Fab) (width 0.1))
     (fp_line (start 3.75 17.05) (end 3.75 18.05) (layer F.Fab) (width 0.1))
+    (fp_text user "PCB Edge" (at 0 -2 90) (layer Dwgs.User)
+      (effects (font (size 1 1) (thickness 0.15)))
+    )
     (pad 1 thru_hole roundrect (at 0 10.16 180) (size 1.4 2.6) (drill oval 0.7 1.9) (layers *.Cu *.Mask) (roundrect_rratio 0.25)
       (net 4 /BANANA+))
@@
     )
     (fp_text value "Banana Jack" (at -2.75 8) (layer F.Fab) hide
-      (effects (font (size 1 1) (thickness 0.15)))
-    )
-    (fp_text user "PCB Edge" (at 0 -2 90) (layer Dwgs.User)
       (effects (font (size 1 1) (thickness 0.15)))
     )
@@
     (fp_line (start 3.75 17.05) (end 4.25 17.05) (layer F.Fab) (width 0.1))
     (fp_line (start 3.75 17.05) (end 3.75 18.05) (layer F.Fab) (width 0.1))
+    (fp_text user "PCB Edge" (at 0 -2 90) (layer Dwgs.User)
+      (effects (font (size 1 1) (thickness 0.15)))
+    )
     (pad 1 thru_hole roundrect (at 0 10.16) (size 1.4 2.6) (drill oval 0.7 1.9) (layers *.Cu *.Mask) (roundrect_rratio 0.25)
       (net 1 /BANANA-))
@@
       (net 2 /BNC-))
   )
-  (gr_text 1.0 (at 150 46) (layer B.SilkS)
+  (gr_text 1.1 (at 150 46) (layer B.SilkS)
     (effects (font (size 1 1) (thickness 0.15)) (justify mirror))
   )
-  (gr_text "1.0\n" (at 158.5 100) (layer B.SilkS)
+  (gr_text 1.1 (at 158.5 100) (layer B.SilkS)
     (effects (font (size 1 1) (thickness 0.15)) (justify mirror))
   )
